Commit message: correct lidar position

File: description/lidar.xacro (robot description, xacro)
@@ -4,5 +4,5 @@
         <parent link="chassis"/>
         <child link="laser_frame"/>
-        <origin xyz="0.08 0 0.18" rpy="0 0 0"/>
+        <origin xyz="0.08 0 0.18" rpy="0 0 3.14159"/>
     </joint>
     <link name="laser_frame">
