Commit message: Change IMU frame id

File: description/imu.xacro (robot description, xacro)
@@ -3,8 +3,8 @@
 <joint name="imu_joint" type="fixed">
     <parent link="base_link"/>
-    <child link="imu_link"/>
+    <child link="imu_frame"/>
     <origin xyz="-0.001 0 0.098"/>
 </joint>
-<link name="imu_link">
+<link name="imu_frame">
     <visual>
         <geometry>
@@ -18,5 +18,5 @@
     </collision>
 </link>
-<gazebo reference="imu_link">
+<gazebo reference="imu_frame">
 <sensor name="imu_sensor" type="imu">
 <plugin filename="libgazebo_ros_imu_sensor.so" name="imu_plugin">

Commit message: imu.xacro aktualisieren

File: description/imu.xacro (robot description, xacro)
@@ -3,8 +3,8 @@
 <joint name="imu_joint" type="fixed">
     <parent link="base_link"/>
-    <child link="imu_frame"/>
+    <child link="imu_link"/>
     <origin xyz="-0.001 0 0.098"/>
 </joint>
-<link name="imu_frame">
+<link name="imu_link">
     <visual>
         <geometry>
@@ -18,5 +18,5 @@
     </collision>
 </link>
-<gazebo reference="imu_frame">
+<gazebo reference="imu_link">
 <sensor name="imu_sensor" type="imu">
 <plugin filename="libgazebo_ros_imu_sensor.so" name="imu_plugin">
